Commit message: Completed check in 1 and 2

File: urdf/robot.xacro (robot description, xacro)
@@ -137,5 +137,5 @@
     <child link="camera_link"/>
     <origin xyz="${chassis_length/2} 0 ${chassis_height/2+camera_height/2}"/>
-  </joint>
+  </joint>trsj
   <gazebo reference="chassis">
     <material>Gazebo/Orange</material>
@@ -143,4 +143,28 @@
   <gazebo reference="camera_link">
     <material>Gazebo/Blue</material>
+     <sensor type="camera" name="camera1">
+      <update_rate>30.0</update_rate>
+      <camera name="head">
+        <horizontal_fov>1.3962634</horizontal_fov>
+        <image>
+          <width>800</width>
+          <height>800</height>
+          <format>R8G8B8</format>
+        </image>
+        <clip>
+          <near>0.02</near>
+          <far>300</far>
+        </clip>
+        <noise>
+        </noise>
+      </camera>
+      <plugin name="camera_controller" filename="libgazebo_ros_camera.so">
+        <alwayson>True</alwayson>
+        <updateRate>0.0</updateRate>
+        <cameraName>robot_cam</cameraName>
+        <imageTopicName>/camera/image_raw</imageTopicName>
+        <cameraInfoTopicName>/camera/camera_info</cameraInfoTopicName>
+      </plugin>
+    </sensor>
   </gazebo>
   <gazebo reference="wheel_FL">
@@ -156,3 +180,18 @@
     <material>Gazebo/Yellow</material>
   </gazebo>
+  <gazebo>
+  <plugin name="skid_steer_drive_controller" filename="libgazebo_ros_skid_steer_drive.so">
+      <robotNamespace>/</robotNamespace>
+      <leftFrontJoint>wheel_FL_joint</leftFrontJoint>
+      <rightFrontJoint>wheel_FR_joint</rightFrontJoint>
+      <leftRearJoint>wheel_RL_joint</leftRearJoint>
+      <rightRearJoint>wheel_RR_joint</rightRearJoint>
+      <wheelSeparation>${chassis_width}</wheelSeparation>
+      <wheelDiameter>${wheel_radius * 2}</wheelDiameter>
+      <robotBaseFrame>chassis</robotBaseFrame>
+      <torque>20</torque>
+      <topicName>cmd_vel</topicName>
+      <broadcastTF>false</broadcastTF>
+    </plugin>
+  </gazebo>
 </robot>
